File: PCB/ergodonk_simple_zero.kicad_sch (KiCad schematic)
At the start: 146 parts, among them J2 4PIN, Q1 TIP120, SW0 SW_PUSH_LED, SW08_RH10 SW_PUSH_LED, SW1 SW_PUSH_LED, SW10 SW_PUSH_LED, SW11 SW_PUSH_LED, SW12 SW_PUSH_LED, SW13 SW_PUSH_LED, SW14 SW_PUSH_LED, SW15 SW_PUSH_LED, SW16 SW_PUSH_LED, SW17 SW_PUSH_LED, SW18_RH10 SW_PUSH_LED, SW2 SW_PUSH_LED, SW20 SW_PUSH_LED, SW21 SW_PUSH_LED, SW22 SW_PUSH_LED, SW23 SW_PUSH_LED, SW24 SW_PUSH_LED, SW25 SW_PUSH_LED, SW26 SW_PUSH_LED, SW27 SW_PUSH_LED, SW28_RH10 SW_PUSH_LED, SW3 SW_PUSH_LED, SW30 SW_PUSH_LED, SW31 SW_PUSH_LED, SW32 SW_PUSH_LED, SW33 SW_PUSH_LED, SW34 SW_PUSH_LED, SW35 SW_PUSH_LED, SW36 SW_PUSH_LED, SW37 SW_PUSH_LED, SW38_RH10 SW_PUSH_LED, SW4 SW_PUSH_LED, SW40 SW_PUSH_LED, SW42 SW_PUSH_LED, SW43 SW_PUSH_LED, SW44 SW_PUSH_LED, SW45 SW_PUSH_LED, SW46 SW_PUSH_LED, SW47 SW_PUSH_LED, SW48_RH10 SW_PUSH_LED, SW5 SW_PUSH_LED, SW50 SW_PUSH_LED, SW51 SW_PUSH_LED, SW52 SW_PUSH_LED, SW53 SW_PUSH_LED, SW54 SW_PUSH_LED, SW55 SW_PUSH_LED, SW56 SW_PUSH_LED, SW57 SW_PUSH_LED, SW58 SW_PUSH_LED, SW6 SW_PUSH_LED, SW7 SW_PUSH_LED

Commit message: Footprint library cleanup
Parts:
- SW0, SW1, SW10, SW11, SW12, SW13, SW14, SW15, SW16, SW17, SW2, SW20, SW21, SW22, SW23, SW24, SW25, SW26, SW3, SW30, SW31, SW32, SW33, SW34, SW35, SW36, SW4, SW42, SW43, SW44, SW45, SW46, SW5, SW50, SW51, SW52, SW53, SW54, SW55, SW56, SW6, SW7: footprint Ergodonk_simple_zero:CherryMX_Choc_Hotswap_ergodonk_simple_zero_56 -> Ergodonk_simple_zero:CherryMX_Choc_Hotswap_ergodonk_simple_zero_DS
